Commit message: Deleting useless files and working X500 model, but without pretty mesh

File: models/X500/urdf/X500_base.urdf.xacro (robot description, xacro)
@@ -6,6 +6,6 @@
   <!-- Body Properties -->
   <xacro:property name="rotor_velocity_slowdown_sim" value="15" />
-  <xacro:property name="mesh_file" value="esferas_simulator/models/kopterworx/meshes/kopterworx_model_simple.dae" /> <!-- Cemig: esferas_simulator/models/kopterworx/meshes/Drone_Cemig_v4_rot.dae -->
-  <xacro:property name="mesh_scale" value="0.1" /> <!-- Cemig: 1.0-->
+  <xacro:property name="mesh_file" value="ardupilot_gazebo/models/kopterworx/meshes/kopterworx_model_simple.dae" />
+  <xacro:property name="mesh_scale" value="0.1" />
   <xacro:property name="prop_scale" value="0.003" />
   <xacro:property name="mass" value="9" />  <!-- [kg] -->
@@ -38,10 +38,5 @@
   </xacro:property>
   <!-- Included URDF Files -->
-  <xacro:include filename="$(find esferas_simulator)/models/util/multirotor_base_two_cams.urdf.xacro" />
-  <!--
-  <xacro:include filename="/root/sim_ws/src/esferas_simulator/models/ball/cable.sdf">
-      <origin xyz="0 0 3" rpy="0 0 0"/>
-  </xacro:include>
-  -->
+  <xacro:include filename="$(find tcc_docker)/models/common/multirotor_base.urdf.xacro" />
   <!-- Instantiate multirotor_base_macro once -->
   <xacro:multirotor_base_macro
